File: single_switch_pcb/single_switch_pcb.kicad_pcb (KiCad board)
At the start: 2 copper layers, 18 x 18 mm, 13 parts, among them J1 Conn_01x01_Female, J2 Conn_01x01_Female, J3 Conn_01x01_Female, J4 Conn_01x01_Female, U1 switchsocket

Commit message: new design, gerber files updated, readme picture gerber sample updated
Parts:
- removed the REF** at (204.5, 96.5)
- removed the REF** at (204.5, 119.4)
- removed the REF** at (181.6, 119.4)
- removed the REF** at (181.6, 96.5)
- added REF**: m1.6hole, hotswapsocket:m1.6hole, F.Cu at (195.6, 95.2)
- added REF**: m1.6hole, hotswapsocket:m1.6hole, F.Cu at (195.6, 110.5)
- added REF**: m1.6hole, hotswapsocket:m1.6hole, F.Cu at (180.3, 110.5)
- added REF**: m1.6hole, hotswapsocket:m1.6hole, F.Cu at (180.3, 95.2)
- moved J3 2.38 mm to (191.8, 110.2)
- moved D1 2.10 mm to (186.5, 110.1)
Routing:
- net Net-(D1-Pad1): track 22.1 -> 21.5 mm
- net Net-(J1-Pad1): track 20.1 -> 20.6 mm
Other:
- outline, holes or cut-outs redrawn
Changed lines of the file:
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@@
     (thickness 1.6)
     (drawings 6)
-    (tracks 25)
+    (tracks 29)
     (zones 0)
     (modules 13)
@@
   )
   (module hotswapsocket:m1.6hole (layer F.Cu)
-    (at 204.47 96.52)
+    (at 195.58 95.25)
     (descr "Through hole straight pin header, 1x01, 2.54mm pitch, single row")
     (tags "Through hole pin header THT 1x01 2.54mm single row")
@@
   )
   (module hotswapsocket:m1.6hole (layer F.Cu)
-    (at 204.47 119.38)
+    (at 195.58 110.49)
     (descr "Through hole straight pin header, 1x01, 2.54mm pitch, single row")
     (tags "Through hole pin header THT 1x01 2.54mm single row")
@@
   )
   (module hotswapsocket:m1.6hole (layer F.Cu)
-    (at 181.61 119.38)
+    (at 180.34 110.49)
     (descr "Through hole straight pin header, 1x01, 2.54mm pitch, single row")
     (tags "Through hole pin header THT 1x01 2.54mm single row")
@@
   )
   (module hotswapsocket:m1.6hole (layer F.Cu)
-    (at 181.61 96.52)
+    (at 180.34 95.25)
     (descr "Through hole straight pin header, 1x01, 2.54mm pitch, single row")
     (tags "Through hole pin header THT 1x01 2.54mm single row")
@@
   )
   (module Connector_PinHeader_2.54mm:PinHeader_1x01_P2.54mm_Vertical (layer F.Cu)
-    (at 194.15 110.2)
+    (at 191.77 110.2)
     (descr "Through hole straight pin header, 1x01, 2.54mm pitch, single row")
     (tags "Through hole pin header THT 1x01 2.54mm single row")
@@
   )
   (module Diode_SMD:D_SOD-123 (layer F.Cu)
-    (at 188.6 110.14 180)
+    (at 186.5 110.14 180)
     (descr SOD-123)
     (tags SOD-123)
@@
     (pad "" np_thru_hole circle (at 3 0.5) (size 3 3) (drill 3) (layers *.Cu *.Mask))
   )
-  (gr_line (start 197.07 111.76) (end 179.07 111.76) (layer Edge.Cuts) (width 0.05))
+  (gr_line (start 197.07 111.98) (end 179.07 111.98) (layer Edge.Cuts) (width 0.05))
   (gr_line (start 179.07 93.98) (end 179.07 111.98) (layer Edge.Cuts) (width 0.05))
   (gr_line (start 197.07 93.98) (end 197.07 111.98) (layer Edge.Cuts) (width 0.05))
-  (gr_text "CARLO CARINO" (at 190.5 119.38) (layer F.SilkS)
+  (gr_text "CARLO \nCARINO" (at 184.2 95.8) (layer F.SilkS)
     (effects (font (size 1 1) (thickness 0.15)))
   )
@@
   (gr_line (start 197.07 93.98) (end 179.07 93.98) (layer Edge.Cuts) (width 0.05))
   (segment (start 181.18 103.73) (end 181.18 104.28) (width 0.25) (layer F.Cu) (net 1))
-  (segment (start 181.18 104.28) (end 185.9 109) (width 0.25) (layer F.Cu) (net 1))
-  (segment (start 185.9 109.09) (end 186.95 110.14) (width 0.25) (layer F.Cu) (net 1))
-  (segment (start 185.9 109) (end 185.9 109.09) (width 0.25) (layer F.Cu) (net 1))
-  (segment (start 194.09 110.14) (end 194.15 110.2) (width 0.25) (layer F.Cu) (net 2))
-  (segment (start 190.25 110.14) (end 194.09 110.14) (width 0.25) (layer F.Cu) (net 2))
+  (segment (start 181.18 103.73) (end 181.18 103.78) (width 0.25) (layer F.Cu) (net 1))
+  (segment (start 184.85 107.45) (end 184.85 110.14) (width 0.25) (layer F.Cu) (net 1))
+  (segment (start 181.18 103.78) (end 184.85 107.45) (width 0.25) (layer F.Cu) (net 1))
   (segment (start 188.8 95.8) (end 190.65 95.8) (width 0.25) (layer F.Cu) (net 2))
   (segment (start 191.065001 96.215001) (end 191.065001 98.665001) (width 0.25) (layer F.Cu) (net 2))
@@
   (segment (start 191.45 102.6) (end 188.85 105.2) (width 0.25) (layer F.Cu) (net 2))
   (segment (start 188.85 105.2) (end 188.85 107.55) (width 0.25) (layer F.Cu) (net 2))
-  (segment (start 190.25 108.95) (end 190.25 110.14) (width 0.25) (layer F.Cu) (net 2))
-  (segment (start 188.85 107.55) (end 190.25 108.95) (width 0.25) (layer F.Cu) (net 2))
-  (via (at 184.75 109.45) (size 0.8) (drill 0.4) (layers F.Cu B.Cu) (net 3))
-  (segment (start 182.7 107.4) (end 184.75 109.45) (width 0.25) (layer F.Cu) (net 3))
-  (segment (start 180.85 107.4) (end 182.7 107.4) (width 0.25) (layer F.Cu) (net 3))
-  (via (at 193.9 108.4) (size 0.8) (drill 0.4) (layers F.Cu B.Cu) (net 3))
-  (segment (start 185.8 108.4) (end 193.9 108.4) (width 0.25) (layer B.Cu) (net 3))
-  (segment (start 184.75 109.45) (end 185.8 108.4) (width 0.25) (layer B.Cu) (net 3))
+  (segment (start 191.71 110.14) (end 191.77 110.2) (width 0.25) (layer F.Cu) (net 2))
+  (segment (start 188.15 110.14) (end 191.71 110.14) (width 0.25) (layer F.Cu) (net 2))
+  (segment (start 188.15 108.25) (end 188.85 107.55) (width 0.25) (layer F.Cu) (net 2))
+  (segment (start 188.15 110.14) (end 188.15 108.25) (width 0.25) (layer F.Cu) (net 2))
   (segment (start 193.9 107.31) (end 194.88 106.33) (width 0.25) (layer F.Cu) (net 3))
-  (segment (start 193.9 108.4) (end 193.9 107.31) (width 0.25) (layer F.Cu) (net 3))
   (segment (start 194.88 104.27) (end 195.75 103.4) (width 0.25) (layer F.Cu) (net 3))
   (segment (start 194.88 106.33) (end 194.88 104.27) (width 0.25) (layer F.Cu) (net 3))
+  (via (at 182.88 107.95) (size 0.8) (drill 0.4) (layers F.Cu B.Cu) (net 3))
+  (segment (start 183.33 108.4) (end 182.88 107.95) (width 0.25) (layer B.Cu) (net 3))
+  (segment (start 185.8 108.4) (end 183.33 108.4) (width 0.25) (layer B.Cu) (net 3))
+  (segment (start 182.88 107.95) (end 182.7 107.77) (width 0.25) (layer F.Cu) (net 3))
+  (segment (start 182.33 107.4) (end 182.88 107.95) (width 0.25) (layer F.Cu) (net 3))
+  (segment (start 180.85 107.4) (end 182.33 107.4) (width 0.25) (layer F.Cu) (net 3))
+  (via (at 193.6 108.3) (size 0.8) (drill 0.4) (layers F.Cu B.Cu) (net 3))
+  (segment (start 194.88 107.02) (end 193.6 108.3) (width 0.25) (layer F.Cu) (net 3))
+  (segment (start 194.88 106.33) (end 194.88 107.02) (width 0.25) (layer F.Cu) (net 3))
+  (segment (start 185.9 108.3) (end 185.8 108.4) (width 0.25) (layer B.Cu) (net 3))
+  (segment (start 193.6 108.3) (end 185.9 108.3) (width 0.25) (layer B.Cu) (net 3))
 )
